Commit message: rviz_plugin package init

File: pneutrunk_description/urdf/segment_macro.xacro (robot description, xacro)
@@ -8,5 +8,5 @@
         <visual>
             <geometry>
-                <cylinder length="0.1" radius="0.3"/>
+                <cylinder length="0.1" radius="0.15"/>
                 <origin rpy="0 0 0" xyz="0 0 0"/>
             </geometry>
