Commit message: init description

File: pneutrunk_description/urdf/pneutrunk.xacro (robot description, xacro)
@@ -2,12 +2,17 @@
 <robot name="pneutrunk" xmlns:xacro="http://www.ros.org/wiki/xacro">
 <!-- TODO: Create base link -->
-<link name="world"/>
+<xacro:include filename="$(find pneutrunk_description)/urdf/pneutrunk_table_macro.xacro"/>
+<xacro:pneutrunk_table />
 <!-- Add robot -->
-<xacro:include filename="$(find pneutrunk_description)/urdf/segment_macro.xacro"/>
-    <xacro:segment suffix="1" base_link="world"/>
-    <xacro:segment suffix="2" base_link="world"/>
-    <xacro:segment suffix="3" base_link="world"/>
-    <xacro:segment suffix="4" base_link="world"/>
-    <xacro:segment suffix="5" base_link="world"/>
-    <xacro:segment suffix="6" base_link="world"/>
+<!-- <xacro:include filename="$(find pneutrunk_description)/urdf/segment_macro.xacro"/>
+<xacro:segment suffix="1" baselink="base_link"/> -->
+<!-- <xacro:segment suffix="2" baselink="base_link"/>
+<xacro:segment suffix="3" baselink="base_link"/>
+<xacro:segment suffix="4" baselink="base_link"/>
+<xacro:segment suffix="5" baselink="base_link"/>
+<xacro:segment suffix="6" baselink="base_link"/>
+<joint name="segment_1_joint" type="fixed">
+    <parent link="base_link"/>
+    <child link="segment_1"/>
+</joint> -->
 </robot>

File: pneutrunk_description/urdf/segment_macro.xacro (robot description, xacro)
@@ -4,6 +4,7 @@
     <color rgba="1 1 1 1"/>
 </material>
-<xacro:macro name="segment" params="suffix base_link">
-    <link name="segment_${suffix}">
+<link name="base_link"/>
+<xacro:macro name="segment" params="suffix baselink">
+    <link name="segment_$(suffix)">
         <visual>
             <geometry>
@@ -14,7 +15,7 @@
         </visual>
     </link>
-    <joint name="segment_${suffix}_joint" type="fixed">
-        <parent link="${base_link}"/>
-        <child link="segment_${suffix}"/>
+    <joint name="segment_$(suffix)_joint" type="fixed">
+        <parent link="$(baselink)"/>
+        <child link="segment_$(suffix)"/>
     </joint>
 </xacro:macro>

Commit message: kinematics template

File: pneutrunk_description/urdf/pneutrunk.xacro (robot description, xacro)
@@ -5,14 +5,10 @@
 <xacro:pneutrunk_table />
 <!-- Add robot -->
-<!-- <xacro:include filename="$(find pneutrunk_description)/urdf/segment_macro.xacro"/>
-<xacro:segment suffix="1" baselink="base_link"/> -->
-<!-- <xacro:segment suffix="2" baselink="base_link"/>
-<xacro:segment suffix="3" baselink="base_link"/>
-<xacro:segment suffix="4" baselink="base_link"/>
-<xacro:segment suffix="5" baselink="base_link"/>
-<xacro:segment suffix="6" baselink="base_link"/>
-<joint name="segment_1_joint" type="fixed">
-    <parent link="base_link"/>
-    <child link="segment_1"/>
-</joint> -->
+ <xacro:include filename="$(find pneutrunk_description)/urdf/segment_macro.xacro"/>
+<xacro:segment id="1" baselink="tool_link"/>
+<xacro:segment id="2" baselink="tool_link"/>
+<xacro:segment id="3" baselink="tool_link"/>
+<xacro:segment id="4" baselink="tool_link"/>
+<xacro:segment id="5" baselink="tool_link"/>
+<xacro:segment id="6" baselink="tool_link"/>
 </robot>

File: pneutrunk_description/urdf/segment_macro.xacro (robot description, xacro)
@@ -4,7 +4,6 @@
     <color rgba="1 1 1 1"/>
 </material>
-<link name="base_link"/>
-<xacro:macro name="segment" params="suffix baselink">
-    <link name="segment_$(suffix)">
+<xacro:macro name="segment" params="id baselink">
+    <link name="segment_${id}">
         <visual>
             <geometry>
@@ -15,7 +14,7 @@
         </visual>
     </link>
-    <joint name="segment_$(suffix)_joint" type="fixed">
-        <parent link="$(baselink)"/>
-        <child link="segment_$(suffix)"/>
+    <joint name="segment_${id}_joint" type="fixed">
+        <parent link="${baselink}"/>
+        <child link="segment_${id}"/>
     </joint>
 </xacro:macro>

Commit message: ForwardKinematics

File: pneutrunk_description/urdf/pneutrunk.xacro (robot description, xacro)
@@ -12,3 +12,4 @@
 <xacro:segment id="5" baselink="tool_link"/>
 <xacro:segment id="6" baselink="tool_link"/>
+<xacro:segment id="7" baselink="tool_link"/>
 </robot>

File: pneutrunk_description/urdf/segment_macro.xacro (robot description, xacro)
@@ -8,5 +8,5 @@
         <visual>
             <geometry>
-                <cylinder length="0.1" radius="0.15"/>
+                <cylinder length="0.025" radius="0.15"/>
                 <origin rpy="0 0 0" xyz="0 0 0"/>
             </geometry>
