Commit message: full stack v1

File: pneutrunk_description/urdf/pneutrunk_table_macro.xacro (robot description, xacro)
@@ -3,27 +3,41 @@
 <xacro:macro name="pneutrunk_table">
     <link name="base_link">
-        <visual>
-        <origin xyz="0 0 0" rpy="0 0 0" />
+        <inertial>
+            <origin
+                xyz="-0.434770940222074 -0.792173144511564 1.62663324904387"
+                rpy="0 0 0" />
+            <mass value="3" />
+        <inertia
+            ixx="1.32651553814696"
+            ixy="0.000517555260969639"
+            ixz="0.0219200370677011"
+            iyy="1.01290522605608"
+            iyz="-0.0177124498363617"
+            izz="0.550947775469309" />
+        </inertial>
+    <visual>
+        <origin
+            xyz="0 0 0"
+            rpy="0 0 0" />
         <geometry>
-            <mesh filename="package://pneutrunk_description/meshes/base.stl" />
+            <mesh filename="package://pneutrunk_description/meshes/base_link.STL" />
         </geometry>
         <material name="">
-            <color rgba="0.792156862745098 0.819607843137255 0.933333333333333 1" />
-        </material>
-        </visual>
+            <color rgba="0.898039215686275 0.917647058823529 0.929411764705882 1" />
+      </material>
+    </visual>
+    <collision>
+        <origin
+            xyz="0 0 0"
+            rpy="0 0 0" />
+        <geometry>
+            <mesh filename="package://pneutrunk_description/meshes/base_link.STL" />
+        </geometry>
+    </collision>
     </link>
-    <link name="tool_link">
-        <visual>
-            <origin xyz="0 0 0" rpy="0 0 0" />
-            <geometry>
-                <mesh filename="package://pneutrunk_description/meshes/tool.stl" />
-            </geometry>
-            <material name="">
-                <color rgba="0.752941176470588 0.752941176470588 0.752941176470588 1" />
-            </material>
-        </visual>
-    </link>
+    <link name="tool_link"/>
     <joint name="base_tool_joint" type="fixed">
-        <origin xyz="-0.42937 -1.001 -0.80522" rpy="0 1.5708 0" />
+        <origin xyz="0.8 0.834121320343554 2.03812132034355"
+                rpy="0 0 0" />
         <parent link="base_link" />
         <child link="tool_link" />

Commit message: gui v1 launch file

File: pneutrunk_description/urdf/pneutrunk_table_macro.xacro (robot description, xacro)
@@ -3,17 +3,4 @@
 <xacro:macro name="pneutrunk_table">
     <link name="base_link">
-        <inertial>
-            <origin
-                xyz="-0.434770940222074 -0.792173144511564 1.62663324904387"
-                rpy="0 0 0" />
-            <mass value="3" />
-        <inertia
-            ixx="1.32651553814696"
-            ixy="0.000517555260969639"
-            ixz="0.0219200370677011"
-            iyy="1.01290522605608"
-            iyz="-0.0177124498363617"
-            izz="0.550947775469309" />
-        </inertial>
     <visual>
         <origin
@@ -27,12 +14,4 @@
       </material>
     </visual>
-    <collision>
-        <origin
-            xyz="0 0 0"
-            rpy="0 0 0" />
-        <geometry>
-            <mesh filename="package://pneutrunk_description/meshes/base_link.STL" />
-        </geometry>
-    </collision>
     </link>
     <link name="tool_link"/>
